Commit message: Modified ee to hand offset, added flange link, and dummy links for planning.

File: iiwa_robotiq_description/urdf/iiwa_robotiq.urdf.xacro (robot description, xacro)
@@ -11,16 +11,11 @@
   <xacro:arg name="hardware_interface" default="PositionJointInterface"/>
   <xacro:arg name="robot_name" default="iiwa"/>
-  <!--  Define the origin of your 3D space
-  Here we define a box lying at 0,0,0 with some dimensions, in reality our robot is place on top of a metal cart with those dimensions.
-  This will include the cart in the scene and avoid the robot to hit it when using MoveIt!
-  If you don't want to have that you can define a basic world link (see commented lines)
-  -->
-  <!--     <link name="world"/> -->
-  <!-- TODO: Adjust table surface dimensions-->
+  <!-- Table surface centered 5 cm below the origin in the z direction. -->
   <link name="world">
     <visual>
       <origin xyz="0 0 -0.05" rpy="0 0 0"/>
       <geometry>
-	<box size="2.5 2.5 0.099"/>
+    <!-- 9.9cm thick so it doesn't intersect with arm model. -->
+    <box size="2.5 2.5 0.099"/>
       </geometry>
     </visual>
@@ -28,5 +23,5 @@
       <origin xyz="0 0 -0.05" rpy="0 0 0"/>
       <geometry>
-	<box size="2.5 2.5 0.099"/>
+    <box size="2.5 2.5 0.099"/>
       </geometry>
     </collision>
@@ -35,20 +30,56 @@
     <static>true</static>
   </gazebo>
-  <!-- Here we insert an iiwa7 robot in the scene, it's origin is just on top of the box previously defined. You can use 0,0,0 if you don't have that. -->
+  <!-- Here we insert an iiwa7 robot in the scene, it's origin is just on top of the box previously defined.-->
   <xacro:iiwa7 hardware_interface="$(arg hardware_interface)" robot_name="$(arg robot_name)" parent="world">
-    <origin xyz="0 0 0.0" rpy="0 0 0"/>
+    <origin xyz="0 0 0" rpy="0 0 0"/>
   </xacro:iiwa7>
-  <!-- TODO -->
+  <!-- Instantiate the robotiq model from the imported macro. -->
   <xacro:robotiq-3f-gripper_articulated prefix="">
   </xacro:robotiq-3f-gripper_articulated>
-  <!-- robotiq properties -->
-  <xacro:property name="robotiq_mass" value="2.3" />
-  <xacro:property name="robotiq_joint_offset" value="0.00 0.00 0.097" />
-  <!--  Here we define a dummy joint between the tip of the iiwa7 and the base of the robotiq.
-  There is no offset between the two, that means the robotiq is attached at the robot flange. -->
+  <!-- Here we define a flange link between the tip of the iiwa7 and the base of the robotiq. -->
+  <!-- Insert a cylinder between default (smaller) flange and robotiq. -->
+  <link name="flange">
+    <visual>
+      <geometry>
+        <!-- Length and radius computed by SGD (Semi-stochastic GraduateStudent Descent). -->
+        <cylinder length="0.037" radius="0.035"/>
+      </geometry>
+      <material name="blue">
+        <color rgba="0 0 .8 1"/>
+      </material>
+    </visual>
+    <collision>
+      <geometry>
+        <cylinder length="0.037" radius="0.035"/>
+      </geometry>
+    </collision>
+  </link>
+  <!-- Link at surface of palm for planning. -->
+  <link name="palm_surface"/>
+  <!-- Link near the center of the grasp region for planning. -->
+  <link name="finger_grasp_centroid"/>
+  <!-- The offset between iiwa_link_ee and palm was estimated to be 0.0975.
+       Sum of z origin displacements of ee_to_flange and robotiq_joint. -->
+  <joint name="ee_to_flange" type="fixed">
+    <parent link="iiwa_link_ee"/>
+    <child link="flange"/>
+    <origin xyz ="0.0 0.0 0.0225"/>
+  </joint>
   <joint name="robotiq_joint" type="fixed">
-    <parent link="iiwa_link_ee" />
+    <parent link="flange" />
     <child link = "palm" />
-    <origin xyz="${robotiq_joint_offset}" rpy="${PI/2.0} 0 ${PI/2.0}" />
+    <origin xyz="0.0 0.0 0.075" rpy="${PI/2.0} 0 ${PI/2.0}" />
+  </joint>
+  <joint name="palm_to_palm_surface" type="fixed">
+    <parent link="palm"/>
+    <child link="palm_surface"/>
+    <!-- Also estimated heuristically. -->
+    <origin xyz ="0.0 0.05 0.0"/>
+  </joint>
+  <joint name="palm_to_finger_grasp_centroid" type="fixed">
+    <parent link="palm"/>
+    <child link="finger_grasp_centroid"/>
+    <!-- Also estimated heuristically. -->
+    <origin xyz ="0.0 0.125 0.0"/>
   </joint>
 </robot>

Commit message: Link between arm and hand is orange instead of blue.

File: iiwa_robotiq_description/urdf/iiwa_robotiq.urdf.xacro (robot description, xacro)
@@ -45,6 +45,6 @@
         <cylinder length="0.037" radius="0.035"/>
       </geometry>
-      <material name="blue">
-        <color rgba="0 0 .8 1"/>
+      <material name="orange">
+        <color rgba="1.0 0.27 0.0 1"/>
       </material>
     </visual>

Commit message: Increased arm-hand link size

File: iiwa_robotiq_description/urdf/iiwa_robotiq.urdf.xacro (robot description, xacro)
@@ -16,6 +16,6 @@
       <origin xyz="0 0 -0.05" rpy="0 0 0"/>
       <geometry>
-    <!-- 9.9cm thick so it doesn't intersect with arm model. -->
-    <box size="2.5 2.5 0.099"/>
+    <!-- 9.99cm thick so it doesn't intersect with arm model. -->
+    <box size="2.5 2.5 0.0999"/>
       </geometry>
     </visual>
@@ -23,5 +23,5 @@
       <origin xyz="0 0 -0.05" rpy="0 0 0"/>
       <geometry>
-    <box size="2.5 2.5 0.099"/>
+    <box size="2.5 2.5 0.0999"/>
       </geometry>
     </collision>
@@ -43,5 +43,5 @@
       <geometry>
         <!-- Length and radius computed by SGD (Semi-stochastic GraduateStudent Descent). -->
-        <cylinder length="0.037" radius="0.035"/>
+        <cylinder length="0.038" radius="0.035"/>
       </geometry>
       <material name="orange">
@@ -51,5 +51,5 @@
     <collision>
       <geometry>
-        <cylinder length="0.037" radius="0.035"/>
+        <cylinder length="0.038" radius="0.035"/>
       </geometry>
     </collision>

Commit message: Use 1.57... instead of  in URDF xacro because Gazebo can't parse.

File: iiwa_robotiq_description/urdf/iiwa_robotiq.urdf.xacro (robot description, xacro)
@@ -69,5 +69,7 @@
     <parent link="flange" />
     <child link = "palm" />
-    <origin xyz="0.0 0.0 0.075" rpy="${PI/2.0} 0 ${PI/2.0}" />
+    <!-- Gazebo isn't happy about ${PI/2.0}-->
+    <!--<origin xyz="0.0 0.0 0.075" rpy="${PI/2.0} 0 ${PI/2.0}" />-->
+    <origin xyz="0.0 0.0 0.075" rpy="1.57079632679 0 1.57079632679" />
   </joint>
   <joint name="palm_to_palm_surface" type="fixed">

Commit message: Added structure sensor frame to robot URDF.

File: iiwa_robotiq_description/urdf/iiwa_robotiq.urdf.xacro (robot description, xacro)
@@ -59,4 +59,6 @@
   <!-- Link near the center of the grasp region for planning. -->
   <link name="finger_grasp_centroid"/>
+  <!-- Link for structure sensor with OpenNI2-->
+  <link name="camera_link"/>
   <!-- The offset between iiwa_link_ee and palm was estimated to be 0.0975.
        Sum of z origin displacements of ee_to_flange and robotiq_joint. -->
@@ -65,4 +67,9 @@
     <child link="flange"/>
     <origin xyz ="0.0 0.0 0.0225"/>
+  </joint>
+  <joint name="ee_to_structure" type="fixed">
+    <parent link="iiwa_link_ee"/>
+    <child link="camera_link"/>
+    <origin xyz ="0.04 -0.08 0.03" rpy="0 0 -1.5707963"/>
   </joint>
   <joint name="robotiq_joint" type="fixed">

Commit message: Added structure sensor model to robot model for collision avoidance.

File: iiwa_robotiq_description/urdf/iiwa_robotiq.urdf.xacro (robot description, xacro)
@@ -55,4 +55,21 @@
     </collision>
   </link>
+  <!-- Structure sensor model -->
+  <link name="structure_sensor_model">
+    <visual>
+      <geometry>
+        <!-- 5" wide, 1" other two dimensions. Surface (x) is at origin -->
+        <box size="0.0254 0.127 0.0254"/>
+      </geometry>
+      <material name="orange">
+        <color rgba="1.0 0.27 0.0 1"/>
+      </material>
+    </visual>
+    <collision>
+      <geometry>
+        <box size="0.0254 0.127 0.0254"/>
+      </geometry>
+    </collision>
+  </link>
   <!-- Link at surface of palm for planning. -->
   <link name="palm_surface"/>
@@ -72,4 +89,10 @@
     <child link="camera_link"/>
     <origin xyz ="0.04 -0.08 0.03" rpy="0 0 -1.5707963"/>
+  </joint>
+  <joint name="structure_to_sensor_model" type="fixed">
+    <parent link="camera_link"/>
+    <child link="structure_sensor_model"/>
+    <!-- x offset half x dim so it's at surface, y to center it-->
+    <origin xyz="-0.0127 -0.04 0" rpy="0 0 0"/>
   </joint>
   <joint name="robotiq_joint" type="fixed">

Commit message: Added boxes in model around cable connections so they're considered during path planning.

File: iiwa_robotiq_description/urdf/iiwa_robotiq.urdf.xacro (robot description, xacro)
@@ -72,4 +72,36 @@
     </collision>
   </link>
+  <!-- Collision model for gripper cable connections -->
+  <link name="gripper_cable_link">
+    <visual>
+      <geometry>
+        <box size="0.0254 0.0254 0.0762"/>
+      </geometry>
+      <material name="orange">
+        <color rgba="1.0 0.27 0.0 1"/>
+      </material>
+    </visual>
+    <collision>
+      <geometry>
+        <box size="0.0254 0.0254 0.0762"/>
+      </geometry>
+    </collision>
+  </link>
+  <!-- Collision model for wrist cable connections -->
+  <link name="wrist_cable_link">
+    <visual>
+      <geometry>
+        <box size="0.0254 0.0254 0.0254"/>
+      </geometry>
+      <material name="orange">
+        <color rgba="1.0 0.27 0.0 1"/>
+      </material>
+    </visual>
+    <collision>
+      <geometry>
+        <box size="0.0254 0.0254 0.0254"/>
+      </geometry>
+    </collision>
+  </link>
   <!-- Link at surface of palm for planning. -->
   <link name="palm_surface"/>
@@ -103,4 +135,14 @@
     <origin xyz="0.0 0.0 0.075" rpy="1.57079632679 0 1.57079632679" />
   </joint>
+  <joint name="palm_to_gripper_cable" type="fixed">
+    <parent link="palm"/>
+    <child link="gripper_cable_link"/>
+    <origin xyz ="0.0927 -0.01 0.0"/>
+  </joint>
+  <joint name="ee_to_wrist_cable" type="fixed">
+    <parent link="iiwa_link_ee"/>
+    <child link="wrist_cable_link"/>
+    <origin xyz ="0.0 0.0727 -0.03"/>
+  </joint>
   <joint name="palm_to_palm_surface" type="fixed">
     <parent link="palm"/>

Commit message: Added mat and object box collision models.

File: iiwa_robotiq_description/urdf/iiwa_robotiq.urdf.xacro (robot description, xacro)
@@ -16,6 +16,6 @@
       <origin xyz="0 0 -0.05" rpy="0 0 0"/>
       <geometry>
-    <!-- 9.99cm thick so it doesn't intersect with arm model. -->
-    <box size="2.5 2.5 0.0999"/>
+        <!-- 9.99cm thick so it doesn't intersect with arm model. -->
+        <box size="2.5 2.5 0.0999"/>
       </geometry>
     </visual>
@@ -23,5 +23,5 @@
       <origin xyz="0 0 -0.05" rpy="0 0 0"/>
       <geometry>
-    <box size="2.5 2.5 0.0999"/>
+        <box size="2.5 2.5 0.0999"/>
       </geometry>
     </collision>
@@ -30,4 +30,37 @@
     <static>true</static>
   </gazebo>
+  <!-- Mat in front of arm - 1cm tall-->
+  <link name="mat">
+    <visual>
+      <origin xyz="0 0 0" rpy="0 0 0"/>
+      <geometry>
+        <box size="1.0 2.5 0.02"/>
+      </geometry>
+    </visual>
+    <collision>
+      <origin xyz="0 0 0.0" rpy="0 0 0"/>
+      <geometry>
+        <box size="1.0 2.5 0.02"/>
+      </geometry>
+    </collision>
+  </link>
+  <link name="obj_box">
+    <visual>
+      <origin xyz="0 0 0" rpy="0 0 0"/>
+      <geometry>
+        <!-- 12" 16" 8.5" -->
+        <box size="0.3048 0.4064 0.2159"/>
+      </geometry>
+      <material name="brown">
+        <color rgba="0.627 0.321 0.176 1"/>
+      </material>
+    </visual>
+    <collision>
+      <origin xyz="0 0 0.0" rpy="0 0 0"/>
+      <geometry>
+        <box size="0.3048 0.4064 0.2159"/>
+      </geometry>
+    </collision>
+  </link>
   <!-- Here we insert an iiwa7 robot in the scene, it's origin is just on top of the box previously defined.-->
   <xacro:iiwa7 hardware_interface="$(arg hardware_interface)" robot_name="$(arg robot_name)" parent="world">
@@ -110,4 +143,18 @@
   <!-- Link for structure sensor with OpenNI2-->
   <link name="camera_link"/>
+  <!-- Mat in front of arm - 17cm from origin in x direction-->
+  <joint name="world_to_mat" type="fixed">
+    <parent link="world"/>
+    <child link="mat"/>
+    <origin xyz ="0.67 0.0 0.0"/>
+  </joint>
+  <!-- 19.25 inches from center to box edge. x, back edge is at 0-->
+  <!-- 0.3048 0.4064 0.2159 -->
+  <joint name="world_to_obj_box" type="fixed">
+    <parent link="world"/>
+    <child link="obj_box"/>
+    <!-- -xdim/2, 19.25" + ydim/2, zdim=2-->
+    <origin xyz ="-0.1524 0.69215 0.10795"/>
+  </joint>
   <!-- The offset between iiwa_link_ee and palm was estimated to be 0.0975.
        Sum of z origin displacements of ee_to_flange and robotiq_joint. -->

Commit message: Updated camera calibration.

File: iiwa_robotiq_description/urdf/iiwa_robotiq.urdf.xacro (robot description, xacro)
@@ -167,5 +167,5 @@
     <parent link="iiwa_link_ee"/>
     <child link="camera_link"/>
-    <origin xyz ="0.04 -0.08 0.03" rpy="0 0 -1.5707963"/>
+    <origin xyz ="0.049 -0.082 0.03" rpy="0 0 -1.5707963"/>
   </joint>
   <joint name="structure_to_sensor_model" type="fixed">

Commit message: Increase size of box, wrist cable.

File: iiwa_robotiq_description/urdf/iiwa_robotiq.urdf.xacro (robot description, xacro)
@@ -50,5 +50,6 @@
       <geometry>
         <!-- 12" 16" 8.5" -->
-        <box size="0.3048 0.4064 0.2159"/>
+        <!-- Real z: 0.2159 -->
+        <box size="0.3048 0.4064 0.3"/>
       </geometry>
       <material name="brown">
@@ -59,5 +60,5 @@
       <origin xyz="0 0 0.0" rpy="0 0 0"/>
       <geometry>
-        <box size="0.3048 0.4064 0.2159"/>
+        <box size="0.3048 0.4064 0.3"/>
       </geometry>
     </collision>
@@ -125,13 +126,13 @@
     <visual>
       <geometry>
-        <box size="0.0254 0.0254 0.0254"/>
-      </geometry>
-      <material name="orange">
-        <color rgba="1.0 0.27 0.0 1"/>
-      </material>
-    </visual>
-    <collision>
-      <geometry>
-        <box size="0.0254 0.0254 0.0254"/>
+        <box size="0.0254 0.0354 0.0254"/>
+      </geometry>
+      <material name="orange">
+        <color rgba="1.0 0.27 0.0 1"/>
+      </material>
+    </visual>
+    <collision>
+      <geometry>
+        <box size="0.0254 0.0354 0.0254"/>
       </geometry>
     </collision>
@@ -154,6 +155,6 @@
     <parent link="world"/>
     <child link="obj_box"/>
-    <!-- -xdim/2, 19.25" + ydim/2, zdim=2-->
-    <origin xyz ="-0.1524 0.69215 0.10795"/>
+    <!-- -xdim/2, 19.25" + ydim/2, zdim/2-->
+    <origin xyz ="-0.1524 0.69215 0.15"/>
   </joint>
   <!-- The offset between iiwa_link_ee and palm was estimated to be 0.0975.
@@ -190,5 +191,6 @@
     <parent link="iiwa_link_ee"/>
     <child link="wrist_cable_link"/>
-    <origin xyz ="0.0 0.0727 -0.03"/>
+    <!-- Link extended by 0.01 in y direction - offset from 0.0727 to ...-->
+    <origin xyz ="0.0 0.0777 -0.03"/>
   </joint>
   <joint name="palm_to_palm_surface" type="fixed">

Commit message: Revert model changes, too difficult to plan to goals, there's clearance..

File: iiwa_robotiq_description/urdf/iiwa_robotiq.urdf.xacro (robot description, xacro)
@@ -50,6 +50,5 @@
       <geometry>
         <!-- 12" 16" 8.5" -->
-        <!-- Real z: 0.2159 -->
-        <box size="0.3048 0.4064 0.3"/>
+        <box size="0.3048 0.4064 0.2159"/>
       </geometry>
       <material name="brown">
@@ -60,5 +59,5 @@
       <origin xyz="0 0 0.0" rpy="0 0 0"/>
       <geometry>
-        <box size="0.3048 0.4064 0.3"/>
+        <box size="0.3048 0.4064 0.2159"/>
       </geometry>
     </collision>
@@ -126,13 +125,13 @@
     <visual>
       <geometry>
-        <box size="0.0254 0.0354 0.0254"/>
-      </geometry>
-      <material name="orange">
-        <color rgba="1.0 0.27 0.0 1"/>
-      </material>
-    </visual>
-    <collision>
-      <geometry>
-        <box size="0.0254 0.0354 0.0254"/>
+        <box size="0.0254 0.0254 0.0254"/>
+      </geometry>
+      <material name="orange">
+        <color rgba="1.0 0.27 0.0 1"/>
+      </material>
+    </visual>
+    <collision>
+      <geometry>
+        <box size="0.0254 0.0254 0.0254"/>
       </geometry>
     </collision>
@@ -155,6 +154,6 @@
     <parent link="world"/>
     <child link="obj_box"/>
-    <!-- -xdim/2, 19.25" + ydim/2, zdim/2-->
-    <origin xyz ="-0.1524 0.69215 0.15"/>
+    <!-- -xdim/2, 19.25" + ydim/2, zdim=2-->
+    <origin xyz ="-0.1524 0.69215 0.10795"/>
   </joint>
   <!-- The offset between iiwa_link_ee and palm was estimated to be 0.0975.
@@ -191,6 +190,5 @@
     <parent link="iiwa_link_ee"/>
     <child link="wrist_cable_link"/>
-    <!-- Link extended by 0.01 in y direction - offset from 0.0727 to ...-->
-    <origin xyz ="0.0 0.0777 -0.03"/>
+    <origin xyz ="0.0 0.0727 -0.03"/>
   </joint>
   <joint name="palm_to_palm_surface" type="fixed">

Commit message: Color the table in the URDF to match the scene and for visibility.

File: iiwa_robotiq_description/urdf/iiwa_robotiq.urdf.xacro (robot description, xacro)
@@ -19,4 +19,7 @@
         <box size="2.5 2.5 0.0999"/>
       </geometry>
+      <material name="gray">
+        <color rgba="0.75 0.75 0.75 1"/>
+      </material>
     </visual>
     <collision>
@@ -37,4 +40,7 @@
         <box size="1.0 2.5 0.02"/>
       </geometry>
+      <material name="black">
+        <color rgba="0.0 0.0 0.0 1"/>
+      </material>
     </visual>
     <collision>

Commit message: Increased size of camera model in arm URDF to avoid collisions and close calls.

File: iiwa_robotiq_description/urdf/iiwa_robotiq.urdf.xacro (robot description, xacro)
@@ -99,13 +99,14 @@
       <geometry>
         <!-- 5" wide, 1" other two dimensions. Surface (x) is at origin -->
-        <box size="0.0254 0.127 0.0254"/>
-      </geometry>
-      <material name="orange">
-        <color rgba="1.0 0.27 0.0 1"/>
-      </material>
-    </visual>
-    <collision>
-      <geometry>
-        <box size="0.0254 0.127 0.0254"/>
+        <!-- x increase .01, y increase .1, z increase 0.005 -->
+        <box size="0.0324 0.137 0.0304"/>
+      </geometry>
+      <material name="orange">
+        <color rgba="1.0 0.27 0.0 1"/>
+      </material>
+    </visual>
+    <collision>
+      <geometry>
+        <box size="0.0324 0.137 0.0304"/>
       </geometry>
     </collision>
@@ -179,5 +180,6 @@
     <child link="structure_sensor_model"/>
     <!-- x offset half x dim so it's at surface, y to center it-->
-    <origin xyz="-0.0127 -0.04 0" rpy="0 0 0"/>
+    <!--<origin xyz="-0.0127 -0.04 0" rpy="0 0 0"/>-->
+    <origin xyz="-0.0162 -0.05 0" rpy="0 0 0"/>
   </joint>
   <joint name="robotiq_joint" type="fixed">

Commit message: Increase boundary around power cable connector on wrist.

File: iiwa_robotiq_description/urdf/iiwa_robotiq.urdf.xacro (robot description, xacro)
@@ -132,13 +132,14 @@
     <visual>
       <geometry>
-        <box size="0.0254 0.0254 0.0254"/>
-      </geometry>
-      <material name="orange">
-        <color rgba="1.0 0.27 0.0 1"/>
-      </material>
-    </visual>
-    <collision>
-      <geometry>
-        <box size="0.0254 0.0254 0.0254"/>
+        <!--<box size="0.0254 0.0254 0.0254"/>-->
+        <box size="0.03 0.03 0.0254"/>
+      </geometry>
+      <material name="orange">
+        <color rgba="1.0 0.27 0.0 1"/>
+      </material>
+    </visual>
+    <collision>
+      <geometry>
+        <box size="0.03 0.03 0.0254"/>
       </geometry>
     </collision>

Commit message: Bring box model 2" closer to base of robot.

File: iiwa_robotiq_description/urdf/iiwa_robotiq.urdf.xacro (robot description, xacro)
@@ -162,6 +162,6 @@
     <parent link="world"/>
     <child link="obj_box"/>
-    <!-- -xdim/2, 19.25" + ydim/2, zdim=2-->
-    <origin xyz ="-0.1524 0.69215 0.10795"/>
+    <!-- -xdim/2, 19.25" + ydim/2 - 2", zdim=2-->
+    <origin xyz ="-0.1524 0.64135 0.10795"/>
   </joint>
   <!-- The offset between iiwa_link_ee and palm was estimated to be 0.0975.

Commit message: Box model bigger to avoid collisions.

File: iiwa_robotiq_description/urdf/iiwa_robotiq.urdf.xacro (robot description, xacro)
@@ -55,6 +55,6 @@
       <origin xyz="0 0 0" rpy="0 0 0"/>
       <geometry>
-        <!-- 12" 16" 8.5" -->
-        <box size="0.3048 0.4064 0.2159"/>
+        <!-- 12"+ 16" 8.5"+ -->
+        <box size="0.35 0.4064 0.25"/>
       </geometry>
       <material name="brown">

Commit message: adding wall

File: iiwa_robotiq_description/urdf/iiwa_robotiq.urdf.xacro (robot description, xacro)
@@ -33,4 +33,22 @@
     <static>true</static>
   </gazebo>
+  <!-- Table behind wall, arm - 1m back-->
+  <link name="wall">
+    <visual>
+      <origin xyz="0 0 0" rpy="0 0 0"/>
+      <geometry>
+        <box size="0.1 10 5"/>
+      </geometry>
+      <material name="black">
+        <color rgba="0.0 0.0 0.0 1"/>
+      </material>
+    </visual>
+    <collision>
+      <origin xyz="0 0 0.0" rpy="0 0 0"/>
+      <geometry>
+        <box size="1.0 2.5 0.02"/>
+      </geometry>
+    </collision>
+  </link>
   <!-- Mat in front of arm - 1cm tall-->
   <link name="mat">
@@ -157,4 +175,10 @@
     <origin xyz ="0.67 0.0 0.0"/>
   </joint>
+  <!-- wall behind arm-->
+  <joint name="world_to_wall" type="fixed">
+    <parent link="world"/>
+    <child link="wall"/>
+    <origin xyz ="-1 0 0.0"/>
+  </joint>
   <!-- 19.25 inches from center to box edge. x, back edge is at 0-->
   <!-- 0.3048 0.4064 0.2159 -->

Commit message: Fixed wall, arm now avoids collision.

File: iiwa_robotiq_description/urdf/iiwa_robotiq.urdf.xacro (robot description, xacro)
@@ -47,5 +47,5 @@
       <origin xyz="0 0 0.0" rpy="0 0 0"/>
       <geometry>
-        <box size="1.0 2.5 0.02"/>
+        <box size="0.1 10 5"/>
       </geometry>
     </collision>
@@ -179,5 +179,5 @@
     <parent link="world"/>
     <child link="wall"/>
-    <origin xyz ="-1 0 0.0"/>
+    <origin xyz ="-0.8 0 0.0"/>
   </joint>
   <!-- 19.25 inches from center to box edge. x, back edge is at 0-->
