Commit message: Replace box for dropping object with cabinet.

File: iiwa_robotiq_description/urdf/iiwa_robotiq.urdf.xacro (robot description, xacro)
@@ -69,10 +69,11 @@
     </collision>
   </link>
-  <link name="obj_box">
-    <visual>
-      <origin xyz="0 0 0" rpy="0 0 0"/>
-      <geometry>
-        <!-- 12"+ 16" 8.5"+ -->
-        <box size="0.35 0.4064 0.25"/>
+  <!-- Box for dropping objects, to the left of the arm -->
+  <!-- 12"+ 16" 8.5"+ -->
+  <!--<link name="obj_box">
+    <visual>
+      <origin xyz="0 0 0" rpy="0 0 0"/>
+      <geometry>
+        <box size="0.3048 0.4064 0.2159"/>
       </geometry>
       <material name="brown">
@@ -84,4 +85,22 @@
       <geometry>
         <box size="0.3048 0.4064 0.2159"/>
+      </geometry>
+    </collision>
+  </link>-->
+  <!-- 30" tall, 38" from origin to surface in x, left side is 3" out into y, 17.5" wide, 12.5" deep -->
+  <link name="cabinet">
+    <visual>
+      <origin xyz="0 0 0" rpy="0 0 0"/>
+      <geometry>
+        <box size="0.3175 0.4445 0.762"/>
+      </geometry>
+      <material name="brown">
+        <color rgba="0.627 0.321 0.176 1"/>
+      </material>
+    </visual>
+    <collision>
+      <origin xyz="0 0 0.0" rpy="0 0 0"/>
+      <geometry>
+        <box size="0.3175 0.4445 0.762"/>
       </geometry>
     </collision>
@@ -183,9 +202,15 @@
   <!-- 19.25 inches from center to box edge. x, back edge is at 0-->
   <!-- 0.3048 0.4064 0.2159 -->
-  <joint name="world_to_obj_box" type="fixed">
+  <!-- origin: -xdim/2, 19.25" + ydim/2 - 2", zdim=2-->
+  <!--<joint name="world_to_obj_box" type="fixed">
     <parent link="world"/>
     <child link="obj_box"/>
-    <!-- -xdim/2, 19.25" + ydim/2 - 2", zdim=2-->
     <origin xyz ="-0.1524 0.64135 0.10795"/>
+  </joint>-->
+  <!-- 30" tall, 38" from origin to surface in x, left side is 3" out into y, 17.5" wide, 12.5" deep -->
+  <joint name="world_to_cabinet" type="fixed">
+    <parent link="world"/>
+    <child link="cabinet"/>
+    <origin xyz ="1.12395 -0.14605 0.381"/>
   </joint>
   <!-- The offset between iiwa_link_ee and palm was estimated to be 0.0975.

Commit message: Moved cabinet closer to arm, increased height to 1m.

File: iiwa_robotiq_description/urdf/iiwa_robotiq.urdf.xacro (robot description, xacro)
@@ -93,5 +93,5 @@
       <origin xyz="0 0 0" rpy="0 0 0"/>
       <geometry>
-        <box size="0.3175 0.4445 0.762"/>
+        <box size="0.3175 0.4445 1.0"/>
       </geometry>
       <material name="brown">
@@ -102,5 +102,5 @@
       <origin xyz="0 0 0.0" rpy="0 0 0"/>
       <geometry>
-        <box size="0.3175 0.4445 0.762"/>
+        <box size="0.3175 0.4445 1.0"/>
       </geometry>
     </collision>
@@ -208,9 +208,9 @@
     <origin xyz ="-0.1524 0.64135 0.10795"/>
   </joint>-->
-  <!-- 30" tall, 38" from origin to surface in x, left side is 3" out into y, 17.5" wide, 12.5" deep -->
+  <!-- 30" tall, 36.75" from origin to surface in x, left side is 3" out into y, 17.5" wide, 12.5" deep -->
   <joint name="world_to_cabinet" type="fixed">
     <parent link="world"/>
     <child link="cabinet"/>
-    <origin xyz ="1.12395 -0.14605 0.381"/>
+    <origin xyz ="1.0922 -0.14605 0.5"/>
   </joint>
   <!-- The offset between iiwa_link_ee and palm was estimated to be 0.0975.

Commit message: Added blocks to URDF.

File: iiwa_robotiq_description/urdf/iiwa_robotiq.urdf.xacro (robot description, xacro)
@@ -89,5 +89,12 @@
   </link>-->
   <!-- 30" tall, 38" from origin to surface in x, left side is 3" out into y, 17.5" wide, 12.5" deep -->
+  <!-- Blocks: 10.5" from center to edge negative y.-->
+  <!--         z from 4 to 8, then another 14" to 18"-->
+  <!--         3.5" into x, 7 for whole rack-->
+  <!--         3.5" wide (y) -->
+  <!--         y_org in world: 10.5+3.5/2= 12.25-->
+  <!--         y_org in door: 12.25-(17.5/2-3)=6.5 -->
   <link name="cabinet">
+    <!-- Main cabinet -->
     <visual>
       <origin xyz="0 0 0" rpy="0 0 0"/>
@@ -103,4 +110,36 @@
       <geometry>
         <box size="0.3175 0.4445 1.0"/>
+      </geometry>
+    </collision>
+    <!-- Handle blocks lower -->
+    <visual>
+      <origin xyz="-0.24765 -0.1651 -0.3476" rpy="0 0 0"/>
+      <geometry>
+        <box size="0.1778 0.0889 0.1016"/>
+      </geometry>
+      <material name="brown">
+        <color rgba="0.627 0.321 0.176 1"/>
+      </material>
+    </visual>
+    <collision>
+      <origin xyz="-0.24765 -0.1651 -0.3476" rpy="0 0 0"/>
+      <geometry>
+        <box size="0.1778 0.0889 0.1016"/>
+      </geometry>
+    </collision>
+    <!-- Handle blocks upper -->
+    <visual>
+      <origin xyz="-0.24765 -0.1651 0.1096" rpy="0 0 0"/>
+      <geometry>
+        <box size="0.1778 0.0889 0.1016"/>
+      </geometry>
+      <material name="brown">
+        <color rgba="0.627 0.321 0.176 1"/>
+      </material>
+    </visual>
+    <collision>
+      <origin xyz="-0.24765 -0.1651 0.1096" rpy="0 0 0"/>
+      <geometry>
+        <box size="0.1778 0.0889 0.1016"/>
       </geometry>
     </collision>

Commit message: Move cabinet model closer to deter collisions.

File: iiwa_robotiq_description/urdf/iiwa_robotiq.urdf.xacro (robot description, xacro)
@@ -247,9 +247,9 @@
     <origin xyz ="-0.1524 0.64135 0.10795"/>
   </joint>-->
-  <!-- 30" tall, 36.75" from origin to surface in x, left side is 3" out into y, 17.5" wide, 12.5" deep -->
+  <!-- 30" tall, 38" (we use 34.75") from origin to surface in x, left side is 3" out into y, 17.5" wide, 12.5" deep -->
   <joint name="world_to_cabinet" type="fixed">
     <parent link="world"/>
     <child link="cabinet"/>
-    <origin xyz ="1.0922 -0.14605 0.5"/>
+    <origin xyz ="1.0414 -0.14605 0.5"/>
   </joint>
   <!-- The offset between iiwa_link_ee and palm was estimated to be 0.0975.

Commit message: Increase width of cabinet to deter collisions.

File: iiwa_robotiq_description/urdf/iiwa_robotiq.urdf.xacro (robot description, xacro)
@@ -88,5 +88,5 @@
     </collision>
   </link>-->
-  <!-- 30" tall, 38" from origin to surface in x, left side is 3" out into y, 17.5" wide, 12.5" deep -->
+  <!-- 30" tall, 38" from origin to surface in x, left side is 3" out into y, 17.5" + 8.5"padding wide, 12.5" deep -->
   <!-- Blocks: 10.5" from center to edge negative y.-->
   <!--         z from 4 to 8, then another 14" to 18"-->
@@ -100,5 +100,5 @@
       <origin xyz="0 0 0" rpy="0 0 0"/>
       <geometry>
-        <box size="0.3175 0.4445 1.0"/>
+        <box size="0.3175 0.6604 1.0"/>
       </geometry>
       <material name="brown">
@@ -109,5 +109,5 @@
       <origin xyz="0 0 0.0" rpy="0 0 0"/>
       <geometry>
-        <box size="0.3175 0.4445 1.0"/>
+        <box size="0.3175 0.6604 1.0"/>
       </geometry>
     </collision>

Commit message: Added handle to cabinet model.

File: iiwa_robotiq_description/urdf/iiwa_robotiq.urdf.xacro (robot description, xacro)
@@ -112,4 +112,18 @@
       </geometry>
     </collision>
+    <!-- Handle -->
+    <!-- 29" from origin to outer bit of noodle, 2.25 wide - 10.375" x from origin w/ 41" x origin-->
+    <!-- z origin halfway between blocks -->
+    <visual>
+      <origin xyz="-0.263525 -0.1651 -0.119" rpy="0 0 0"/>
+      <geometry>
+        <cylinder length="0.4572" radius="0.028575"/>
+      </geometry>
+      <material name="brown">
+        <color rgba="0.627 0.321 0.176 1"/>
+      </material>
+    </visual>
+    <collision>
+    </collision>
     <!-- Handle blocks lower -->
     <visual>

Commit message: Added collision block.

File: iiwa_robotiq_description/urdf/iiwa_robotiq.urdf.xacro (robot description, xacro)
@@ -125,4 +125,8 @@
     </visual>
     <collision>
+      <origin xyz="-0.263525 -0.1651 -0.119" rpy="0 0 0"/>
+      <geometry>
+        <cylinder length="0.4572" radius="0.028575"/>
+      </geometry>
     </collision>
     <!-- Handle blocks lower -->

Commit message: Remove handle, we'll add it dynamically when needed.

File: iiwa_robotiq_description/urdf/iiwa_robotiq.urdf.xacro (robot description, xacro)
@@ -115,5 +115,6 @@
     <!-- 29" from origin to outer bit of noodle, 2.25 wide - 10.375" x from origin w/ 41" x origin-->
     <!-- z origin halfway between blocks -->
-    <visual>
+    <!-- We're gonna make this a collision object. -->
+    <!--<visual>
       <origin xyz="-0.263525 -0.1651 -0.119" rpy="0 0 0"/>
       <geometry>
@@ -129,5 +130,21 @@
         <cylinder length="0.4572" radius="0.028575"/>
       </geometry>
-    </collision>
+    </collision>-->
+    <!-- Equivalent box for testing purposes -->
+    <!--<visual>
+      <origin xyz="-0.263525 -0.1651 -0.119" rpy="0 0 0"/>
+      <geometry>
+        <box size="0.05715 0.05715 0.4572"/>
+      </geometry>
+      <material name="brown">
+        <color rgba="0.627 0.321 0.176 1"/>
+      </material>
+    </visual>
+    <collision>
+      <origin xyz="-0.263525 -0.1651 -0.119" rpy="0 0 0"/>
+      <geometry>
+        <box size="0.05715 0.05715 0.4572"/>
+      </geometry>
+    </collision>-->
     <!-- Handle blocks lower -->
     <visual>

Commit message: Updated cabinet pose based on moved cabinet and point cloud visualized in rviz.

File: iiwa_robotiq_description/urdf/iiwa_robotiq.urdf.xacro (robot description, xacro)
@@ -117,64 +117,64 @@
     <!-- We're gonna make this a collision object. -->
     <!--<visual>
-      <origin xyz="-0.263525 -0.1651 -0.119" rpy="0 0 0"/>
-      <geometry>
-        <cylinder length="0.4572" radius="0.028575"/>
-      </geometry>
-      <material name="brown">
-        <color rgba="0.627 0.321 0.176 1"/>
-      </material>
-    </visual>
-    <collision>
-      <origin xyz="-0.263525 -0.1651 -0.119" rpy="0 0 0"/>
-      <geometry>
-        <cylinder length="0.4572" radius="0.028575"/>
+      <origin xyz="-0.31115 -0.18415 -0.119" rpy="0 0 0"/>
+      <geometry>
+        <cylinder length="0.4572" radius="0.04445"/>
+      </geometry>
+      <material name="brown">
+        <color rgba="0.627 0.321 0.176 1"/>
+      </material>
+    </visual>
+    <collision>
+      <origin xyz="-0.31115 -0.18415 -0.119" rpy="0 0 0"/>
+      <geometry>
+        <cylinder length="0.4572" radius="0.04445"/>
       </geometry>
     </collision>-->
     <!-- Equivalent box for testing purposes -->
     <!--<visual>
-      <origin xyz="-0.263525 -0.1651 -0.119" rpy="0 0 0"/>
-      <geometry>
-        <box size="0.05715 0.05715 0.4572"/>
-      </geometry>
-      <material name="brown">
-        <color rgba="0.627 0.321 0.176 1"/>
-      </material>
-    </visual>
-    <collision>
-      <origin xyz="-0.263525 -0.1651 -0.119" rpy="0 0 0"/>
-      <geometry>
-        <box size="0.05715 0.05715 0.4572"/>
+      <origin xyz="-0.3175 -0.18415 -0.119" rpy="0 0 0"/>
+      <geometry>
+        <box size="0.0889 0.0889 0.4572"/>
+      </geometry>
+      <material name="brown">
+        <color rgba="0.627 0.321 0.176 1"/>
+      </material>
+    </visual>
+    <collision>
+      <origin xyz="-0.3175 -0.18415 -0.119" rpy="0 0 0"/>
+      <geometry>
+        <box size="0.0889 0.0889 0.4572"/>
       </geometry>
     </collision>-->
     <!-- Handle blocks lower -->
     <visual>
-      <origin xyz="-0.24765 -0.1651 -0.3476" rpy="0 0 0"/>
-      <geometry>
-        <box size="0.1778 0.0889 0.1016"/>
-      </geometry>
-      <material name="brown">
-        <color rgba="0.627 0.321 0.176 1"/>
-      </material>
-    </visual>
-    <collision>
-      <origin xyz="-0.24765 -0.1651 -0.3476" rpy="0 0 0"/>
-      <geometry>
-        <box size="0.1778 0.0889 0.1016"/>
+      <origin xyz="-0.24765 -0.18415 -0.3476" rpy="0 0 0"/>
+      <geometry>
+        <box size="0.1778 0.1143 0.1143"/>
+      </geometry>
+      <material name="brown">
+        <color rgba="0.627 0.321 0.176 1"/>
+      </material>
+    </visual>
+    <collision>
+      <origin xyz="-0.24765 -0.18415 -0.3476" rpy="0 0 0"/>
+      <geometry>
+        <box size="0.1778 0.1143 0.1143"/>
       </geometry>
     </collision>
     <!-- Handle blocks upper -->
     <visual>
-      <origin xyz="-0.24765 -0.1651 0.1096" rpy="0 0 0"/>
-      <geometry>
-        <box size="0.1778 0.0889 0.1016"/>
-      </geometry>
-      <material name="brown">
-        <color rgba="0.627 0.321 0.176 1"/>
-      </material>
-    </visual>
-    <collision>
-      <origin xyz="-0.24765 -0.1651 0.1096" rpy="0 0 0"/>
-      <geometry>
-        <box size="0.1778 0.0889 0.1016"/>
+      <origin xyz="-0.24765 -0.18415 0.1096" rpy="0 0 0"/>
+      <geometry>
+        <box size="0.1778 0.1143 0.1143"/>
+      </geometry>
+      <material name="brown">
+        <color rgba="0.627 0.321 0.176 1"/>
+      </material>
+    </visual>
+    <collision>
+      <origin xyz="-0.24765 -0.18415 0.1096" rpy="0 0 0"/>
+      <geometry>
+        <box size="0.1778 0.1143 0.1143"/>
       </geometry>
     </collision>
@@ -286,5 +286,6 @@
     <parent link="world"/>
     <child link="cabinet"/>
-    <origin xyz ="1.0414 -0.14605 0.5"/>
+    <!--xyz ="1.0414 -0.14605 0.5"-->
+    <origin xyz ="1.143 -0.0508 0.5" rpy="0 0 0.418"/>
   </joint>
   <!-- The offset between iiwa_link_ee and palm was estimated to be 0.0975.

Commit message: Adding obstacles to the planning scene isn't working, add cylinder handle back in.

File: iiwa_robotiq_description/urdf/iiwa_robotiq.urdf.xacro (robot description, xacro)
@@ -116,5 +116,5 @@
     <!-- z origin halfway between blocks -->
     <!-- We're gonna make this a collision object. -->
-    <!--<visual>
+    <visual>
       <origin xyz="-0.31115 -0.18415 -0.119" rpy="0 0 0"/>
       <geometry>
@@ -130,5 +130,5 @@
         <cylinder length="0.4572" radius="0.04445"/>
       </geometry>
-    </collision>-->
+    </collision>
     <!-- Equivalent box for testing purposes -->
     <!--<visual>

Commit message: Remove fixed handle from cabinet, it's added to MoveIt.

File: iiwa_robotiq_description/urdf/iiwa_robotiq.urdf.xacro (robot description, xacro)
@@ -116,5 +116,5 @@
     <!-- z origin halfway between blocks -->
     <!-- We're gonna make this a collision object. -->
-    <visual>
+    <!--<visual>
       <origin xyz="-0.31115 -0.18415 -0.119" rpy="0 0 0"/>
       <geometry>
@@ -130,5 +130,5 @@
         <cylinder length="0.4572" radius="0.04445"/>
       </geometry>
-    </collision>
+    </collision>-->
     <!-- Equivalent box for testing purposes -->
     <!--<visual>

Commit message: Updated cabinet pose.

File: iiwa_robotiq_description/urdf/iiwa_robotiq.urdf.xacro (robot description, xacro)
@@ -287,5 +287,5 @@
     <child link="cabinet"/>
     <!--xyz ="1.0414 -0.14605 0.5"-->
-    <origin xyz ="1.143 -0.0508 0.5" rpy="0 0 0.418"/>
+    <origin xyz ="1.0 -0.36 0.5" rpy="0 0 0.418"/>
   </joint>
   <!-- The offset between iiwa_link_ee and palm was estimated to be 0.0975.
